File: main.brd (EAGLE design)
At the start: 85.1 x 40.3 mm, 8 parts, among them X1 1751248, X2 1751251

Commit message: v2
Parts:
- added X3, X4, X5: 1751251, con-phoenix-350:1751251
- renumbered U$1 to SN74A
Connections:
- net LDATA renamed LDATA2
- removed net HDATA: SN74A.6, X2.2
- new net HDATA1: SN74A.3, X2.2
- new net HDATA2: SN74A.6, X3.2
- new net HDATA3: SN74A.8, X4.2
- new net HDATA4: SN74A.12, X5.2
- new net LDATA1: MS1.19, SN74A.2
- new net LDATA3: MS1.21, SN74A.9
- new net LDATA4: MS1.22, SN74A.11
- net +12V: now also X3.3, X4.3, X5.3
- net GND: now also X3.1, X4.1, X5.1
Routing:
- net +12V: track 0.00 -> 174.5 mm, vias 0 -> 1
- net HDATA2: track 0.00 -> 111.8 mm
- net LDATA4: track 0.00 -> 38.9 mm
- net LDATA1: track 0.00 -> 33.1 mm
- net GND: track 104.8 -> 137.9 mm
- net LDATA3: track 0.00 -> 31.3 mm
- net HDATA: track 18.5 -> 0.00 mm
- net HDATA3: track 0.00 -> 17.5 mm
- net HDATA4: track 0.00 -> 14.9 mm
- net HDATA1: track 0.00 -> 10.7 mm
- net +5V: track 67.0 -> 68.3 mm
Other:
- board size 85.1 x 40.3 mm -> 85.1 x 45.4 mm
- board text added: "+12V"
- board text added: "+5V"
- board text added: "DATA 1"
- board text added: "DATA 2"
- board text added: "DATA 3"
- board text added: "DATA 4"
- board text added: "GND"
